File: wig150g.kicad_sch (KiCad schematic)
At the start: 131 parts, among them M1 Fan, SW1 StickOrTig (Stick default), SW2 ToggleOrSwitch for Pedal (Tog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

Commit message: fix typo
Parts:
- R?: symbol wedasLibary:SDS_S3-24V -> wedasLibrary:SDS_S3-24V
- SW1, SW2: symbol wedasLibary:Switch -> wedasLibrary:Switch
- U?: symbol wedasLibary:Transformer_1P_3S -> wedasLibrary:Transformer_1P_3S
- U?: symbol wedasLibary:SDS_S4_24V -> wedasLibrary:SDS_S4_24V
- U?: symbol wedasLibary:Switch2 -> wedasLibrary:Switch2
- U?: symbol wedasLibary:DS2E-MS2-DC24V -> wedasLibrary:DS2E-MS2-DC24V
- U?: symbol wedasLibary:SDS-VS5-24V -> wedasLibrary:SDS-VS5-24V
Changed lines of the file:
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@@
     (pin "2")
   )
-  (symbol (lib_id "wedasLibary:Transformer_1P_3S") (at 74.93 68.58 0) (unit 1)
+  (symbol (lib_id "wedasLibrary:Transformer_1P_3S") (at 74.93 68.58 0) (unit 1)
     (in_bom yes) (on_board yes) (fields_autoplaced)
     (property "Reference" "U?" (id 0) (at 74.93 55.88 0))
@@
     (pin "2")
   )
-  (symbol (lib_name "Switch_1") (lib_id "wedasLibary:Switch") (at 43.18 381 0) (unit 1)
+  (symbol (lib_name "Switch_1") (lib_id "wedasLibrary:Switch") (at 43.18 381 0) (unit 1)
     (in_bom yes) (on_board yes)
     (property "Reference" "SW1" (id 0) (at 48.26 363.22 0)
@@
     (pin "2")
   )
-  (symbol (lib_id "wedasLibary:SDS_S3-24V") (at 224.79 146.05 0) (unit 1)
+  (symbol (lib_id "wedasLibrary:SDS_S3-24V") (at 224.79 146.05 0) (unit 1)
     (in_bom yes) (on_board yes)
     (property "Reference" "R?" (id 0) (at 252.73 157.48 0)
@@
     (pin "2")
   )
-  (symbol (lib_name "Switch_1") (lib_id "wedasLibary:Switch") (at 140.97 381 0) (unit 1)
+  (symbol (lib_name "Switch_1") (lib_id "wedasLibrary:Switch") (at 140.97 381 0) (unit 1)
     (in_bom yes) (on_board yes)
     (property "Reference" "SW2" (id 0) (at 146.05 363.22 0)
@@
     (pin "2")
   )
-  (symbol (lib_id "wedasLibary:SDS_S4_24V") (at 210.82 143.51 0) (unit 1)
+  (symbol (lib_id "wedasLibrary:SDS_S4_24V") (at 210.82 143.51 0) (unit 1)
     (in_bom yes) (on_board yes)
     (property "Reference" "U?" (id 0) (at 234.95 121.92 0)
@@
     (pin "2")
   )
-  (symbol (lib_name "Switch2_1") (lib_id "wedasLibary:Switch2") (at 200.66 383.54 0) (unit 1)
+  (symbol (lib_name "Switch2_1") (lib_id "wedasLibrary:Switch2") (at 200.66 383.54 0) (unit 1)
     (in_bom yes) (on_board yes)
     (property "Reference" "U?" (id 0) (at 200.66 367.03 0)
@@
     (pin "2")
   )
-  (symbol (lib_id "wedasLibary:DS2E-MS2-DC24V") (at 100.33 167.64 0) (unit 1)
+  (symbol (lib_id "wedasLibrary:DS2E-MS2-DC24V") (at 100.33 167.64 0) (unit 1)
     (in_bom yes) (on_board yes)
     (property "Reference" "U?" (id 0) (at 78.74 151.1299 0)
@@
     (pin "2")
   )
-  (symbol (lib_id "wedasLibary:SDS-VS5-24V") (at 157.48 156.21 270) (unit 1)
+  (symbol (lib_id "wedasLibrary:SDS-VS5-24V") (at 157.48 156.21 270) (unit 1)
     (in_bom yes) (on_board yes)
     (property "Reference" "U?" (id 0) (at 170.18 154.9399 90)

Commit message: small fixes
Parts:
- removed C? (x2): 500nF, symbol Device:C
- removed D?: D, symbol Device:D
- removed L?: L_Ferrite, symbol Device:L_Ferrite
- removed R?: 100Ohm 25W, symbol Device:R
- removed R?: Trimmer, symbol Device:R_Variable
- removed R?: 39kOhm, symbol Device:R
- added ArValve: L_Iron, symbol Device:L_Iron
- added C? (x2): 500nF, symbol Device:C
- added C?: C, symbol Device:C
- added C? (x4): 1uF, symbol Device:C
- added D?: D, symbol Device:D
- added J?: Female Socket, symbol Connector:DIN-5
- added J?: Male Cable Connector, symbol Connector:DIN-5
- added L?: Transformer2, symbol Device:L_Iron
- added R?: Trimmer, symbol Device:R_Trim
- added R? (x2): 33Ohm, symbol Device:R
- added R?: 39kOhm, symbol Device:R
- added R?: 100Ohm 25W, symbol Device:R
- added RV?: Foot_Pedal_Poti, symbol Device:R_Potentiometer
- added SW?: Handle_Push, symbol Switch:SW_Push
- D? (x3): value D -> D_Flyback
- R?: symbol wedasLibrary:SDS_S3-24V -> wedasLibary:SDS_S3-24V
- SW1, SW2: symbol wedasLibrary:Switch -> wedasLibary:Switch
- SW? (x3): value OvertempSW -> OvTempSw
- SW?: value SW_DPST -> FrontPwSw
- U?: symbol wedasLibrary:Transformer_1P_3S -> wedasLibary:Transformer_1P_3S
- U?: symbol wedasLibrary:SDS_S4_24V -> wedasLibary:SDS_S4_24V
- U?: value PedalOrPoti (Pedal default) -> PedalEnable (pedal disabled default); symbol wedasLibrary:Switch2 -> wedasLibary:Switch2
- U?: symbol wedasLibrary:DS2E-MS2-DC24V -> wedasLibary:DS2E-MS2-DC24V
- U?: symbol wedasLibrary:SDS-VS5-24V -> wedasLibary:SDS-VS5-24V
Connections:
- net pedal pin 4 is gone; now on net External Poti V+: R?.2
- net thyristorOut is gone; now on net CtrlBrdRef: RV?.1
- net Argon_Valve_1: no longer D?.1 (K), D?.1 (K), U?.11
- net Argon_Valve_2: no longer D?.2 (A), Q?.2 (C)
- net CtrlBrdRef: now also R?.1, R?.2, R?.2; no longer C?.2, D?.2 (A), R?.2, U?.1 (+)
- net CurrentSetBrd: no longer J?.7 (Pin_7), R?.1, U?.8
- net CurrentSetPot: no longer C?.2, RV?.2, U?.9
- net Electrode -: now also C?.1, L?.2, R?.2
- net HF_B: now also L?.1
- net HVreedDisable_Use: now also C?.2, C?.2, J?.2
- net HalfWaveDetect: now also R?.1
- net V- contrlBoard: no longer R?.1, R?.2
- net at C?.2: now also D?.1 (A), D?.1 (K), U?.4
- net at D?.2 (A), D?.2 (A): now also R?.2; no longer R?.1
- net at C?.1, D?.1 (A), D?.1 (K)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: now also C?.1, C?.2
- net at C?.1, R?.2, U?.2 (-): now also D?.1 (K)
- net at D?.2 (A), R?.1: now also R?.1; no longer R?.2
- net at C?.1, U?.3: now also R?.2
- net at U?.1 (+): no longer U?.3
- net HandSwitch_Overwrite renamed TorchSwitch_Overwrite
- net HandleSwitchToggle renamed TorchSwitchToggle
- net HandleSwitch_Latch renamed TorchSwitch_Latch
- net Pedal Pin 1 renamed TorchSwitch
- net TorchSwitch: now also J?.1
- net Pedal Pin 3 renamed Internal Poti V+
- net Internal Poti V+: now also C?.2, J?.3, R?.1
- net Pedal Pin 4 renamed External Poti V+
- net External Poti V+: now also C?.2, J?.4
- new net: ArValve.1, D?.1 (K), D?.1 (K), U?.11
- new net: ArValve.2, D?.2 (A), Q?.2 (C)
- new net: C?.2, R?.1
- new net: C?.1, C?.1, C?.1, C?.1, C?.2
- new net: J?.4, RV?.1, RV?.2
- new net: J?.3, RV?.3
- new net: J?.1, SW?.1
- new net: J?.2, SW?.2
- new net: C?.1, R?.1
- new net CurrentSetTToCtrl: J?.7 (Pin_7), R?.1, U?.8
- new net CurrentSetToRel: C?.2, R?.2, RV?.2, U?.9
- new net Vc controlBoard: C?.2, D?.2 (A), D?.2 (A), R?.1, R?.2, R?.2, U?.1 (+)
- no-connect marks 8 -> 12
Other:
- note added: ""- / --" Switch"
- note added: ""N / F" Switch"
- note added: ""WIG / Elektrode" Switch"
- note added: "10k foot_poti + min setting = half front poti current"
- note added: "20k foot_poti + min setting = quater front poti current"
- note added: "5 Pin Connector"
- note added: "Arc starter EGT Zündgerät WIG dc/Plasma"
- note added: "Current Potentiometer (0 - 150 A)"
- note added: "Optional Pedal and Torch Switch"
- note added: "Red Status Lamp"
- note added: "WIMA RC filter"
- note added: "min resitance = max front poti set current max resistance = zero current"
- note added: "non inverting amplifyer gain 1.39"
- note removed: "Current Potentiometer"
- note removed: "arc starter EGT Zündgerät WIG dc/Plasma"
- moved on the sheet: R_Shunt

Commit message: improve layout and fix zener
Parts:
- removed C?: 91nF, symbol Device:C
- removed D? (x6): D, symbol Device:D
- removed D?: D_Zener, symbol Device:D_Zener
- added C?: 91nF, symbol Device:C
- added D (x2), D?: D_Zener, symbol Device:D_Zener
- added D (x3): 12V, symbol Device:D_Zener
- added D?: D, symbol Device:D
- C_tantal: renamed from C?; value tantal -> 1uF
- D: renamed from D?; value D_Zener -> 12V
- R?: value Trimmer -> Trimmer 3.8kOhm
- RV?: value R_Potentiometer -> Trim Val: 38kOhm
- gave numbers to parts that had none: 1
Connections:
- net Vc controlBoard is gone; now on net GNDA: C?.2, R?.1, R?.2, R?.2, U?.1 (+)
- net External Poti V+: now also U?.1; no longer U?.2
- net Internal Poti V+: now also U?.2; no longer U?.1
- net at R?.1, R?.1: now also D.1 (K)
- net at D?.1 (A), D?.1 (K), U?.4: now also C?.2
- net at C?.1, C?.2, D?.1 (A)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: now also C?.1
- net at C_tantal.2, Q?.3 (G), R?.1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: now also D.2 (A)
- net at C?.1, R?.2, U?.2 (-): now also D?.1 (K)
- net at Q?.2 (D): now also D.1 (K) (x2)
- net at Q?.3 (G), R?.1, R?.1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: now also D.2 (A)
- net at D?.1 (K), R?.1, R?.1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: now also R?.1; no longer R?.2
- net at U?.2 (-), U?.2 (-), U?.3: now also R?.2; no longer R?.1
- net at C?.1, R?.1, R?.2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: now also D.1 (K), D?.2 (A)
- net at U?.1 (+): now also U?.3
- net at D.1 (K): now also D.2 (A)
- net CtrlBrdRef renamed GNDA
- net GNDA: now also D.1 (K), D.2 (A), D.2 (A), D?.2 (A); no longer J?.5 (Pin_5)
- net V+ contrlBoard renamed V+ CtrlB
- net V+ CtrlB: now also D?.1 (K)
- net V- contrlBoard renamed -24V
- new net CtrlBrdGnd: J?.5 (Pin_5)
Other:
- note added: "comparator with after rise/fall current"
- note added: "current rise and fall slope circuit"
- note added: "diode limiter and high frequency filter"
- note added: "inverting half wave rectifier with gain"
- note added: "opamp buffer"
- note removed: "buffer"
